File: schematics/fusedoctor.kicad_pcb (KiCad board)
At the start: 2 copper layers, 75 x 60 mm, 39 parts, among them J1 Parallel data, J2 Parallel control, J3 HV serial, J4 Power In, J5 MCU control, Q1 BC547, U1 ATtiny2313A, U2 74HC595, U3 ATtiny13/13V, U4 ATtiny24/44/84, U5 ATmega48A/88A/168A/328, U6 ATtiny2313A/4313A

Commit message: Update silkscreen on schematics
Parts:
- U5: value ATmega48A/88A/168A/328 -> ATmega48*/88*/168*/328*
Changed lines of the file:
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@@
       (effects (font (size 1 1) (thickness 0.15)))
     )
-    (fp_text value ATmega48A/88A/168A/328 (at 4 16.52 90) (layer F.Fab)
+    (fp_text value "ATmega48*/88*/168*/328*" (at 4 16.52 90) (layer F.Fab)
       (effects (font (size 1 1) (thickness 0.15)))
     )
@@
     (fp_line (start 9.15 34.65) (end 9.15 -1.6) (layer F.CrtYd) (width 0.05))
     (fp_line (start 9.15 -1.6) (end -1.55 -1.6) (layer F.CrtYd) (width 0.05))
-    (fp_text user "ATmega48A/88A/168A/328\nATmega48PA/88PA/168PA/328P" (at 4 16.52 90) (layer B.SilkS)
+    (fp_text user "ATmega48*/88*/168*/328*\nATtiny28L/28V/48/88" (at 4 16.52 90) (layer B.SilkS)
       (effects (font (size 1 1) (thickness 0.15)) (justify mirror))
     )
